Commit message: Updated max velocity limits and effort for the arms of reemc

File: reemc_description/urdf/arm/arm.urdf.xacro (robot description, xacro)
@@ -15,8 +15,8 @@
   <xacro:property name="arm_friction"       value="1.0" />
   <xacro:property name="arm_damping"        value="1.0" />
-  <xacro:property name="arm_1_max_vel"      value="5.4" />
-  <xacro:property name="arm_2_max_vel"      value="4.12" />
-  <xacro:property name="arm_3_max_vel"      value="5.15" />
-  <xacro:property name="arm_4_max_vel"      value="5.15" />
+  <xacro:property name="arm_1_max_vel"      value="2.7" />
+  <xacro:property name="arm_2_max_vel"      value="3.66" />
+  <xacro:property name="arm_3_max_vel"      value="4.58" />
+  <xacro:property name="arm_4_max_vel"      value="4.58" />
   <xacro:property name="arm_1_max_effort"   value="44.64" />
   <xacro:property name="arm_2_max_effort"   value="22.32" />

File: reemc_description/urdf/arm/wrist.urdf.xacro (robot description, xacro)
@@ -14,6 +14,10 @@
   <xacro:property name="wrist_friction"       value="1.0" />
   <xacro:property name="wrist_damping"        value="1.0" />
-  <xacro:property name="wrist_max_vel"      value="1.77" />
-  <xacro:property name="wrist_max_effort"   value="3.32" />
+  <xacro:property name="wrist_1_max_vel"      value="1.95" />
+  <xacro:property name="wrist_2_max_vel"      value="1.76" />
+  <xacro:property name="wrist_3_max_vel"      value="1.76" />
+  <xacro:property name="wrist_1_max_effort"   value="3" />
+  <xacro:property name="wrist_2_max_effort"   value="6.6" />
+  <xacro:property name="wrist_3_max_effort"   value="6.6" />
   <xacro:property name="wrist_eps"          value="0.02" />
   <!-- TODO: Update dynamic models -->
@@ -50,5 +54,5 @@
       <origin xyz="-0.088 0.02 0" rpy="0 ${-90.0 * reflect * deg_to_rad} 0" />
       <axis xyz="0 0 1" />
-      <limit lower="${-120.0 * deg_to_rad}" upper="${120.0 * deg_to_rad}" effort="${wrist_max_effort}" velocity="${wrist_max_vel}" /> <!--TODO: Check effort value!-->
+      <limit lower="${-120.0 * deg_to_rad}" upper="${120.0 * deg_to_rad}" effort="${wrist_1_max_effort}" velocity="${wrist_1_max_vel}" /> <!--TODO: Check effort value!-->
       <dynamics friction="${wrist_friction}" damping="${wrist_damping}"/>
       <safety_controller k_position="20"
@@ -85,5 +89,5 @@
       <origin xyz="0 0 ${0.15 * reflect}" rpy="${-90.0 * reflect * deg_to_rad} 0 0" />
       <axis xyz="0 0 1" />
-      <limit lower="${-90.0 * deg_to_rad}" upper="${90.0 * deg_to_rad}" effort="${wrist_max_effort}" velocity="${wrist_max_vel}" />
+      <limit lower="${-90.0 * deg_to_rad}" upper="${90.0 * deg_to_rad}" effort="${wrist_2_max_effort}" velocity="${wrist_2_max_vel}" />
       <dynamics friction="${wrist_friction}" damping="${wrist_damping}"/>
       <safety_controller k_position="20"
@@ -121,5 +125,5 @@
       <origin xyz="0 0 0" rpy="${90.0 * reflect * deg_to_rad} 0 0" />
       <axis xyz="0 0 1" />
-      <limit lower="${-120.0 * deg_to_rad}" upper="${120.0 * deg_to_rad}" effort="${wrist_max_effort}" velocity="${wrist_max_vel}" />
+      <limit lower="${-120.0 * deg_to_rad}" upper="${120.0 * deg_to_rad}" effort="${wrist_3_max_effort}" velocity="${wrist_3_max_vel}" />
       <dynamics friction="${wrist_friction}" damping="${wrist_damping}"/>
       <safety_controller k_position="20"

File: reemc_description/urdf/hand/hand.urdf.xacro (robot description, xacro)
@@ -235,7 +235,7 @@
         <origin xyz="0 0 0" rpy="0 0 0" />
         <mass value="0.01" /> <!-- matrix below must not be zero, or Gazebo won't load -->
-        <inertia ixx="0.1" ixy="0.0" ixz="0.0"
-                 iyy="0.1" iyz="0.0"
-                 izz="0.1" />
+        <inertia ixx="0.00001" ixy="0.0" ixz="0.0"
+                 iyy="0.00001" iyz="0.0"
+                 izz="0.00001" />
       </inertial>
     </link>
